File: IndustrialShield.kicad_pcb (KiCad board)
At the start: 2 copper layers, 74 x 80 mm, 54 parts, among them J1 Screw_Terminal_01x02, J10 Screw_Terminal_01x02, J2 Viola Connector, J3 Screw_Terminal_01x02, J4 Screw_Terminal_01x02, J5 Screw_Terminal_01x02, J6 Screw_Terminal_01x02, J7 Screw_Terminal_01x02, J8 Screw_Terminal_01x02, J9 Screw_Terminal_01x02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

Commit message: setting some component values
Parts:
- removed C8: C_Small, Capacitor_SMD:C_0603_1608Metric_Pad1.05x0.95mm_HandSolder
- removed D3: D_Small, Diode_SMD:D_0805_2012Metric_Pad1.15x1.40mm_HandSolder
- removed Q1, Q2: BC817, Package_TO_SOT_SMD:SOT-23_Handsoldering
- removed R17, R5, R7: 4K7, Resistor_SMD:R_0805_2012Metric_Pad1.15x1.40mm_HandSolder
- removed R18, R19: 8K2, Resistor_SMD:R_0805_2012Metric_Pad1.15x1.40mm_HandSolder
- removed R21: 1K, Resistor_SMD:R_0805_2012Metric_Pad1.15x1.40mm_HandSolder
- removed R6: 10K, Resistor_SMD:R_0805_2012Metric_Pad1.15x1.40mm_HandSolder
- added C3: C_Small, Capacitor_SMD:C_0603_1608Metric_Pad1.05x0.95mm_HandSolder, F.Cu at (155.7, 61.6)
- added D12: LED_Small, LED_SMD:LED_0805_2012Metric_Pad1.15x1.40mm_HandSolder, F.Cu at (136.9, 61.8)
- added K1: G5Q-1A, Relay_THT:Relay_SPST_Omron-G5Q-1A, F.Cu at (207.6, 32.7)
- added K2: G5Q-1A, Relay_THT:Relay_SPST_Omron-G5Q-1A, F.Cu at (207.6, 20.1)
- added R1: 330R, Resistor_SMD:R_0805_2012Metric_Pad1.15x1.40mm_HandSolder, F.Cu at (241.8, 11.5)
- added U1: LM2596S-5.0, Package_TO_SOT_SMD:TO-263-5_TabPin3, F.Cu at (143.3, 16.2)
- D11: value LED_Small -> D_Small; footprint LED_SMD:LED_0805_2012Metric_Pad1.15x1.40mm_HandSolder -> Diode_SMD:D_0805_2012Metric_Pad1.15x1.40mm_HandSolder
- R20: value 1K -> 330R
- R3: value 330R -> 4K7
- R4: value 10K -> 330R
- moved J9 182.0 mm to (192.2, 17.0)
- moved U5 180.4 mm to (229.8, 12.1)
- moved D9 171.1 mm to (230.3, 20.8)
- moved J7 167.4 mm to (180.0, 17.0)
- moved J8 149.7 mm to (174.5, 31.0)
- moved J3 142.4 mm to (155.5, 17.0)
- moved J5 142.3 mm to (167.7, 17.0)
- moved J6 120.8 mm to (162.3, 31.0)
- moved J10 114.8 mm to (186.8, 31.0)
- moved D11 108.2 mm to (141.7, 61.8)
- moved R4 105.5 mm to (151.2, 61.8)
- moved J1 105.1 mm to (137.8, 29.4)
- moved J4 103.7 mm to (150.1, 31.0)
- moved R3 97.2 mm to (146.4, 61.8)
- moved U7 95.0 mm to (148.0, 53.2)
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Connections:
- D11 pad 1: GND -> Net-(C3-Pad1)
- D11 pad 2: Net-(D11-Pad2) -> /input/In2_N
- D9 pad 1: Net-(C8-Pad1) -> +24V
- D9 pad 2: /input/In2_N -> Net-(D9-Pad2)
- J2 pad 1: Net-(J2-Pad1) -> +5V
- J2 pad 4: Net-(J2-Pad4) -> +3V3
- R2 pad 2: +3V3 -> GND
- R3 pad 1: Net-(R3-Pad1) -> Net-(C3-Pad1)
- R3 pad 2: +3V3 -> /input/In2_P
- R4 pad 1: +24V -> Net-(D12-Pad2)
- R4 pad 2: Net-(R4-Pad2) -> SODIMM_103
- U4 pad 1: Net-(R2-Pad1) -> SODIMM_135
- U4 pad 2: SODIMM_135 -> Net-(R2-Pad1)
- U4 pad 4: Net-(Q1-Pad1) -> GND_24V
- U4 pad 5: Net-(R4-Pad2) -> Net-(D2-Pad2)
- U5 pad 1: Net-(R3-Pad1) -> SODIMM_133
- U5 pad 2: SODIMM_133 -> Net-(R1-Pad1)
- U5 pad 4: Net-(Q2-Pad1) -> GND_24V
- U5 pad 5: Net-(R6-Pad2) -> Net-(D9-Pad2)
- U6 pad 4: GND -> SODIMM_98
- U6 pad 5: SODIMM_98 -> +3V3
- U7 pad 1: Net-(C8-Pad1) -> Net-(C3-Pad1)
- U7 pad 4: GND -> SODIMM_103
- U7 pad 5: SODIMM_103 -> +3V3
Routing:
- net (no net): vias 0 -> 4
Other:
- outline, holes or cut-outs redrawn
